Commit message: evol(urdf): fix scaling
Signed-off-by: Mael-RABOT <mael.rabot@epitech.eu>

File: InMoov/urdf/InMoov.urdf (robot description, URDF)
Before this commit: robot InMoov, 16 links, 15 joints
Links:
- link base_node: geometry visual mesh filename=../meshes/stl/stand.stl scale=1.00000 1.00000 1.00000
- link left_shoulder_z_link: geometry visual mesh filename=../meshes/stl/G-__564753.001.stl scale=1.00000 1.00000 1.00000; visual mesh filename=../meshes/stl/G-__564753.002.stl scale=1.00000 1.00000 1.00000
- link right_shoulder_z_link: geometry visual mesh filename=../meshes/stl/G-__566220.001.stl scale=1.00000 1.00000 1.00000; visual mesh filename=../meshes/stl/G-__566220.002.stl scale=1.00000 1.00000 1.00000

Commit message: evol(neck): change link name
Signed-off-by: Mael-RABOT <mael.rabot@epitech.eu>

File: InMoov/urdf/InMoov.urdf (robot description, URDF)
Before this commit: robot InMoov, 16 links, 15 joints
Links:
- removed link i01.head.rollNeck_link
- added link neck_link; visual mesh filename=../meshes/stl/Texture.015.stl scale=1.00000 1.00000 1.00000; visual mesh filename=../meshes/stl/Texture.083.stl scale=1.00000 1.00000 1.00000
Joints:
- joint i01.head.rollNeck_link_joint: child i01.head.rollNeck_link -> neck_link

Commit message: feat(urdf): add working foundation
Signed-off-by: Mael-RABOT <mael.rabot@epitech.eu>

File: InMoov/urdf/InMoov.urdf (robot description, URDF)
Before this commit: robot InMoov, 16 links, 15 joints
Links:
- added link i01.head.eyeLeft_link; visual mesh filename=../meshes/stl/Texture.011.stl scale=1.00000 1.00000 1.00000
- added link i01.head.eyeRight_link; visual mesh filename=../meshes/stl/Texture.012.stl scale=1.00000 1.00000 1.00000
- added link i01.head.jaw_link; visual mesh filename=../meshes/stl/Texture.014.stl scale=1.00000 1.00000 1.00000; visual mesh filename=../meshes/stl/Texture.086.stl scale=1.00000 1.00000 1.00000
- added link i01.leftHand.index2_link; visual mesh filename=../meshes/stl/Texture.019.stl scale=1.00000 1.00000 1.00000
- added link i01.leftHand.index3_link; visual mesh filename=../meshes/stl/Texture.020.stl scale=1.00000 1.00000 1.00000
- added link i01.leftHand.index_link; visual mesh filename=../meshes/stl/Texture.018.stl scale=1.00000 1.00000 1.00000
- added link i01.leftHand.majeure2_link; visual mesh filename=../meshes/stl/Texture.023.stl scale=1.00000 1.00000 1.00000
- added link i01.leftHand.majeure3_link; visual mesh filename=../meshes/stl/Texture.024.stl scale=1.00000 1.00000 1.00000
- added link i01.leftHand.majeure_link; visual mesh filename=../meshes/stl/Texture.022.stl scale=1.00000 1.00000 1.00000
- added link i01.leftHand.pinky0_link; visual mesh filename=../meshes/stl/Texture.041.stl scale=1.00000 1.00000 1.00000
- added link i01.leftHand.pinky2_link; visual mesh filename=../meshes/stl/Texture.028.stl scale=1.00000 1.00000 1.00000
- added link i01.leftHand.pinky3_link; visual mesh filename=../meshes/stl/Texture.029.stl scale=1.00000 1.00000 1.00000
- added link i01.leftHand.pinky_link; visual mesh filename=../meshes/stl/Texture.027.stl scale=1.00000 1.00000 1.00000
- added link i01.leftHand.ringFinger_link; visual mesh filename=../meshes/stl/Texture.032.stl scale=1.00000 1.00000 1.00000
- added link i01.leftHand.ringfinger0_link; visual mesh filename=../meshes/stl/Texture.040.stl scale=1.00000 1.00000 1.00000
- added link i01.leftHand.ringfinger2_link; visual mesh filename=../meshes/stl/Texture.033.stl scale=1.00000 1.00000 1.00000
- added link i01.leftHand.ringfinger3_link; visual mesh filename=../meshes/stl/Texture.034.stl scale=1.00000 1.00000 1.00000
- added link i01.leftHand.thumb1_link; visual mesh filename=../meshes/stl/Texture.035.stl scale=1.00000 1.00000 1.00000
- added link i01.leftHand.thumb3_link; visual mesh filename=../meshes/stl/Texture.038.stl scale=1.00000 1.00000 1.00000
- added link i01.leftHand.thumb_link; visual mesh filename=../meshes/stl/Texture.037.stl scale=1.00000 1.00000 1.00000
- added link i01.leftHand.wrist.001_link; visual mesh filename=../meshes/stl/Texture.235.stl scale=1.00000 1.00000 1.00000
- added link i01.rightHand.index2_link; visual mesh filename=../meshes/stl/Texture.045.stl scale=1.00000 1.00000 1.00000
- added link i01.rightHand.index3_link; visual mesh filename=../meshes/stl/Texture.046.stl scale=1.00000 1.00000 1.00000
- added link i01.rightHand.index_link; visual mesh filename=../meshes/stl/Texture.044.stl scale=1.00000 1.00000 1.00000
- added link i01.rightHand.majeure2_link; visual mesh filename=../meshes/stl/Texture.049.stl scale=1.00000 1.00000 1.00000
- added link i01.rightHand.majeure3_link; visual mesh filename=../meshes/stl/Texture.050.stl scale=1.00000 1.00000 1.00000
- added link i01.rightHand.majeure_link; visual mesh filename=../meshes/stl/Texture.048.stl scale=1.00000 1.00000 1.00000
- added link i01.rightHand.pinky0_link; visual mesh filename=../meshes/stl/Texture.067.stl scale=1.00000 1.00000 1.00000
- added link i01.rightHand.pinky2_link; visual mesh filename=../meshes/stl/Texture.054.stl scale=1.00000 1.00000 1.00000
- added link i01.rightHand.pinky3_link; visual mesh filename=../meshes/stl/Texture.055.stl scale=1.00000 1.00000 1.00000
- added link i01.rightHand.pinky_link; visual mesh filename=../meshes/stl/Texture.053.stl scale=1.00000 1.00000 1.00000
- added link i01.rightHand.ringFinger_link; visual mesh filename=../meshes/stl/Texture.058.stl scale=1.00000 1.00000 1.00000
- added link i01.rightHand.ringfinger0_link; visual mesh filename=../meshes/stl/Texture.066.stl scale=1.00000 1.00000 1.00000
- added link i01.rightHand.ringfinger2_link; visual mesh filename=../meshes/stl/Texture.059.stl scale=1.00000 1.00000 1.00000
- added link i01.rightHand.ringfinger3_link; visual mesh filename=../meshes/stl/Texture.060.stl scale=1.00000 1.00000 1.00000
- added link i01.rightHand.thumb1_link; visual mesh filename=../meshes/stl/Texture.063.stl scale=1.00000 1.00000 1.00000
- added link i01.rightHand.thumb3_link; visual mesh filename=../meshes/stl/Texture.062.stl scale=1.00000 1.00000 1.00000
- added link i01.rightHand.thumb_link; visual mesh filename=../meshes/stl/Texture.061.stl scale=1.00000 1.00000 1.00000
- added link i01.rightHand.wrist.001_link; visual mesh filename=../meshes/stl/Texture.204.stl scale=1.00000 1.00000 1.00000
- link left_wrist_z_link: geometry visual mesh filename=../meshes/stl/Texture.039.stl scale=1.00000 1.00000 1.00000
- link neck_link: geometry 
- link right_wrist_z_link: geometry visual mesh filename=../meshes/stl/Texture.065.stl scale=1.00000 1.00000 1.00000
Joints:
- added joint i01.head.eyeLeft_link_joint: type revolute, parent neck_link, child i01.head.eyeLeft_link, origin xyz=0.29444 -1.07687 0.62487 rpy=0.00000 0.00000 -0.00000, axis 0.99994 0.00000 0.01111, limit lower=-0.17453 upper=0.17453 effort=0.00000 velocity=0.78540
- added joint i01.head.eyeRight_link_joint: type revolute, parent neck_link, child i01.head.eyeRight_link, origin xyz=-0.29604 -1.08731 0.62487 rpy=0.00000 -0.00000 -0.00000, axis 0.99994 0.00000 0.01111, limit lower=-0.17453 upper=0.17453 effort=0.00000 velocity=0.78540
- added joint i01.head.jaw_link_joint: type revolute, parent neck_link, child i01.head.jaw_link, origin xyz=-0.00876 -0.34673 0.57354 rpy=-0.00000 0.00000 -0.00000, axis 0.99994 0.00000 0.01111, limit lower=0.00000 upper=0.17453 effort=0.00000 velocity=0.78540
- added joint i01.leftHand.index2_link_joint: type revolute, parent i01.leftHand.index_link, child i01.leftHand.index2_link, origin xyz=0.00258 0.34105 0.00685 rpy=-0.00000 0.00000 -0.00000, axis -0.99994 0.00000 0.01111, limit lower=0.00000 upper=1.57080 effort=0.00000 velocity=0.78540
- added joint i01.leftHand.index3_link_joint: type revolute, parent i01.leftHand.index2_link, child i01.leftHand.index3_link, origin xyz=0.00103 0.22697 0.00433 rpy=0.00000 -0.00000 -0.00000, axis -0.99994 0.00000 0.01111, limit lower=0.00000 upper=1.57080 effort=0.00000 velocity=0.78540
- added joint i01.leftHand.index_link_joint: type revolute, parent i01.leftHand.wrist.001_link, child i01.leftHand.index_link, origin xyz=0.32645 -0.01145 -0.94982 rpy=-1.56854 -0.09096 -0.00330, axis -0.99994 0.00000 0.01111, limit lower=0.00000 upper=1.57080 effort=0.00000 velocity=0.78540
- added joint i01.leftHand.majeure2_link_joint: type revolute, parent i01.leftHand.majeure_link, child i01.leftHand.majeure2_link, origin xyz=0.00272 0.35935 0.00722 rpy=-0.00000 -0.00000 0.00000, axis -0.99994 0.00000 0.01111, limit lower=0.00000 upper=1.57080 effort=0.00000 velocity=0.78540
- added joint i01.leftHand.majeure3_link_joint: type revolute, parent i01.leftHand.majeure2_link, child i01.leftHand.majeure3_link, origin xyz=0.00109 0.23915 0.00456 rpy=0.00000 -0.00000 -0.00000, axis -0.99994 0.00000 0.01111, limit lower=0.00000 upper=1.57080 effort=0.00000 velocity=0.78540
- added joint i01.leftHand.majeure_link_joint: type revolute, parent i01.leftHand.wrist.001_link, child i01.leftHand.majeure_link, origin xyz=0.07161 -0.01170 -0.98881 rpy=-1.56854 0.00160 -0.00309, axis -0.99994 0.00000 0.01111, limit lower=0.00000 upper=1.57080 effort=0.00000 velocity=0.78540
- added joint i01.leftHand.pinky0_link_joint: type revolute, parent i01.leftHand.wrist.001_link, child i01.leftHand.pinky0_link, origin xyz=-0.24002 0.00108 -0.35218 rpy=-1.56789 -0.68643 -0.00494, axis 0.00000 -0.99994 0.01111, limit lower=0.00000 upper=1.57080 effort=0.00000 velocity=0.78540
- added joint i01.leftHand.pinky2_link_joint: type revolute, parent i01.leftHand.pinky_link, child i01.leftHand.pinky2_link, origin xyz=0.00225 0.29796 0.00599 rpy=-0.00000 0.00000 -0.00000, axis -0.99994 0.00000 0.01111, limit lower=0.00000 upper=1.57080 effort=0.00000 velocity=0.78540
- added joint i01.leftHand.pinky3_link_joint: type revolute, parent i01.leftHand.pinky2_link, child i01.leftHand.pinky3_link, origin xyz=0.00090 0.19830 0.00378 rpy=-0.00000 -0.00000 -0.00000, axis -0.99994 0.00000 0.01111, limit lower=0.00000 upper=1.57080 effort=0.00000 velocity=0.78540
- added joint i01.leftHand.pinky_link_joint: type revolute, parent i01.leftHand.pinky0_link, child i01.leftHand.pinky_link, origin xyz=-0.43178 0.20489 0.00726 rpy=-0.00000 0.00000 0.94526, axis -0.99994 0.00000 0.01111, limit lower=0.00000 upper=1.57080 effort=0.00000 velocity=0.78540
- added joint i01.leftHand.ringFinger_link_joint: type revolute, parent i01.leftHand.ringfinger0_link, child i01.leftHand.ringFinger_link, origin xyz=-0.33329 0.15280 -0.00664 rpy=-0.00000 0.00000 0.77485, axis -0.99994 0.00000 0.01111, limit lower=0.00000 upper=1.57080 effort=0.00000 velocity=0.78540
- added joint i01.leftHand.ringfinger0_link_joint: type revolute, parent i01.leftHand.wrist.001_link, child i01.leftHand.ringfinger0_link, origin xyz=-0.05673 0.00101 -0.57588 rpy=-1.56789 -0.68643 -0.00494, axis 0.00000 -0.99994 0.01111, limit lower=0.00000 upper=1.57080 effort=0.00000 velocity=0.78540
- added joint i01.leftHand.ringfinger2_link_joint: type revolute, parent i01.leftHand.ringFinger_link, child i01.leftHand.ringfinger2_link, origin xyz=0.00258 0.34105 0.00685 rpy=-0.00000 -0.00000 0.00000, axis -0.99994 0.00000 0.01111, limit lower=0.00000 upper=1.57080 effort=0.00000 velocity=0.78540
- added joint i01.leftHand.ringfinger3_link_joint: type revolute, parent i01.leftHand.ringfinger2_link, child i01.leftHand.ringfinger3_link, origin xyz=0.00103 0.22697 0.00433 rpy=-0.00000 0.00000 -0.00000, axis -0.99994 0.00000 0.01111, limit lower=0.00000 upper=1.57080 effort=0.00000 velocity=0.78540
- added joint i01.leftHand.thumb1_link_joint: type revolute, parent i01.leftHand.wrist.001_link, child i01.leftHand.thumb1_link, origin xyz=0.28234 -0.00002 -0.37340 rpy=1.51635 -0.09893 -0.00332, axis 0.00000 -0.99994 0.01111, limit lower=0.00000 upper=1.57080 effort=0.00000 velocity=0.78540
- added joint i01.leftHand.thumb3_link_joint: type revolute, parent i01.leftHand.thumb_link, child i01.leftHand.thumb3_link, origin xyz=0.01229 -0.33047 -0.00704 rpy=0.00001 -0.00000 0.00000, axis -0.99994 0.00000 0.01111, limit lower=0.00000 upper=1.57080 effort=0.00000 velocity=0.78540
- added joint i01.leftHand.thumb_link_joint: type revolute, parent i01.leftHand.thumb1_link, child i01.leftHand.thumb_link, origin xyz=0.25977 -0.13332 -0.00800 rpy=-0.03182 -0.32566 0.83064, axis -0.99994 0.00000 0.01111, limit lower=0.00000 upper=1.57080 effort=0.00000 velocity=0.78540
- added joint i01.leftHand.wrist.001_link_joint: type revolute, parent left_wrist_z_link, child i01.leftHand.wrist.001_link, origin xyz=-0.00000 -0.00000 -0.16925 rpy=-0.00000 0.00000 -0.61611, axis -0.99994 0.00000 0.01111, limit lower=0.00000 upper=1.57080 effort=0.00000 velocity=0.78540
- added joint i01.rightHand.index2_link_joint: type revolute, parent i01.rightHand.index_link, child i01.rightHand.index2_link, origin xyz=-0.00258 -0.34105 -0.00685 rpy=0.00000 -0.00000 0.00000, axis -0.99994 0.00000 0.01111, limit lower=0.00000 upper=1.57080 effort=0.00000 velocity=0.78540
- added joint i01.rightHand.index3_link_joint: type revolute, parent i01.rightHand.index2_link, child i01.rightHand.index3_link, origin xyz=-0.00103 -0.22697 -0.00432 rpy=0.00000 0.00000 -0.00000, axis -0.99994 0.00000 0.01111, limit lower=0.00000 upper=1.57080 effort=0.00000 velocity=0.78540
- added joint i01.rightHand.index_link_joint: type revolute, parent i01.rightHand.wrist.001_link, child i01.rightHand.index_link, origin xyz=-0.32320 -0.00773 -0.95398 rpy=1.57305 0.09096 -0.01576, axis -0.99994 0.00000 0.01111, limit lower=0.00000 upper=1.57080 effort=0.00000 velocity=0.78540
- added joint i01.rightHand.majeure2_link_joint: type revolute, parent i01.rightHand.majeure_link, child i01.rightHand.majeure2_link, origin xyz=-0.00272 -0.35935 -0.00722 rpy=-0.00000 -0.00000 -0.00000, axis -0.99994 0.00000 0.01111, limit lower=0.00000 upper=1.57080 effort=0.00000 velocity=0.78540
- added joint i01.rightHand.majeure3_link_joint: type revolute, parent i01.rightHand.majeure2_link, child i01.rightHand.majeure3_link, origin xyz=-0.00109 -0.23915 -0.00456 rpy=0.00000 -0.00000 0.00000, axis -0.99994 0.00000 0.01111, limit lower=0.00000 upper=1.57080 effort=0.00000 velocity=0.78540
- added joint i01.rightHand.majeure_link_joint: type revolute, parent i01.rightHand.wrist.001_link, child i01.rightHand.majeure_link, origin xyz=-0.06841 -0.01284 -0.99297 rpy=1.57305 -0.00160 -0.01597, axis -0.99994 0.00000 0.01111, limit lower=0.00000 upper=1.57080 effort=0.00000 velocity=0.78540
- added joint i01.rightHand.pinky0_link_joint: type revolute, parent i01.rightHand.wrist.001_link, child i01.rightHand.pinky0_link, origin xyz=0.24340 -0.00601 -0.35634 rpy=1.57370 0.68643 -0.01412, axis 0.00000 -0.99994 0.01111, limit lower=0.00000 upper=1.57080 effort=0.00000 velocity=0.78540
- added joint i01.rightHand.pinky2_link_joint: type revolute, parent i01.rightHand.pinky_link, child i01.rightHand.pinky2_link, origin xyz=-0.00225 -0.29796 -0.00598 rpy=0.00000 0.00000 -0.00000, axis -0.99994 0.00000 0.01111, limit lower=0.00000 upper=1.57080 effort=0.00000 velocity=0.78540
- added joint i01.rightHand.pinky3_link_joint: type revolute, parent i01.rightHand.pinky2_link, child i01.rightHand.pinky3_link, origin xyz=-0.00090 -0.19830 -0.00378 rpy=0.00000 0.00000 0.00000, axis -0.99994 0.00000 0.01111, limit lower=0.00000 upper=1.57080 effort=0.00000 velocity=0.78540
- added joint i01.rightHand.pinky_link_joint: type revolute, parent i01.rightHand.pinky0_link, child i01.rightHand.pinky_link, origin xyz=0.43178 -0.20489 -0.00726 rpy=-0.00000 -0.00000 0.94526, axis -0.99994 0.00000 0.01111, limit lower=0.00000 upper=1.57080 effort=0.00000 velocity=0.78540
- added joint i01.rightHand.ringFinger_link_joint: type revolute, parent i01.rightHand.ringfinger0_link, child i01.rightHand.ringFinger_link, origin xyz=0.33328 -0.15280 0.00664 rpy=-0.00000 -0.00000 0.77485, axis -0.99994 0.00000 0.01111, limit lower=0.00000 upper=1.57080 effort=0.00000 velocity=0.78540
- added joint i01.rightHand.ringfinger0_link_joint: type revolute, parent i01.rightHand.wrist.001_link, child i01.rightHand.ringfinger0_link, origin xyz=0.06015 -0.00258 -0.58004 rpy=1.57370 0.68643 -0.01412, axis 0.00000 -0.99994 0.01111, limit lower=0.00000 upper=1.57080 effort=0.00000 velocity=0.78540
- added joint i01.rightHand.ringfinger2_link_joint: type revolute, parent i01.rightHand.ringFinger_link, child i01.rightHand.ringfinger2_link, origin xyz=-0.00258 -0.34105 -0.00685 rpy=-0.00000 -0.00000 0.00000, axis -0.99994 0.00000 0.01111, limit lower=0.00000 upper=1.57080 effort=0.00000 velocity=0.78540
- added joint i01.rightHand.ringfinger3_link_joint: type revolute, parent i01.rightHand.ringfinger2_link, child i01.rightHand.ringfinger3_link, origin xyz=-0.00103 -0.22697 -0.00432 rpy=-0.00000 0.00000 -0.00000, axis -0.99994 0.00000 0.01111, limit lower=0.00000 upper=1.57080 effort=0.00000 velocity=0.78540
- added joint i01.rightHand.thumb1_link_joint: type revolute, parent i01.rightHand.wrist.001_link, child i01.rightHand.thumb1_link, origin xyz=-0.27888 0.00285 -0.37757 rpy=-1.62525 0.09893 -0.01574, axis 0.00000 -0.99994 0.01111, limit lower=0.00000 upper=1.57080 effort=0.00000 velocity=0.78540
- added joint i01.rightHand.thumb3_link_joint: type revolute, parent i01.rightHand.thumb_link, child i01.rightHand.thumb3_link, origin xyz=-0.01229 0.33047 0.00704 rpy=0.00001 -0.00000 0.00000, axis -0.99994 0.00000 0.01111, limit lower=0.00000 upper=1.57080 effort=0.00000 velocity=0.78540
- added joint i01.rightHand.thumb_link_joint: type revolute, parent i01.rightHand.thumb1_link, child i01.rightHand.thumb_link, origin xyz=-0.25977 0.13332 0.00800 rpy=-0.03182 -0.32566 0.83064, axis -0.99994 0.00000 0.01111, limit lower=0.00000 upper=1.57080 effort=0.00000 velocity=0.78540
- added joint i01.rightHand.wrist.001_link_joint: type revolute, parent right_wrist_z_link, child i01.rightHand.wrist.001_link, origin xyz=-0.00000 -0.00000 -0.16508 rpy=0.00000 0.00000 0.63517, axis -0.99994 0.00000 0.01111, limit lower=0.00000 upper=1.57080 effort=0.00000 velocity=0.78540
- joint i01.head.rollNeck_link_joint: limit lower=0 upper=0 -> lower=0 upper=0 velocity=0.78540

Commit message: evol(urdf): fix eye angle & add schema
Signed-off-by: Mael-RABOT <mael.rabot@epitech.eu>

File: InMoov/urdf/InMoov.urdf (robot description, URDF)
Before this commit: robot InMoov, 55 links, 54 joints
Links:
- link left_shoulder_x_link: geometry visual mesh filename=../meshes/stl/Texture.003.stl scale=1.00000 1.00000 1.00000; visual mesh filename=../meshes/stl/Texture.254.stl scale=1.00000 1.00000 1.00000
- link neck_link: geometry visual mesh filename=../meshes/stl/Texture.015.stl scale=1.00000 1.00000 1.00000; visual mesh filename=../meshes/stl/Texture.083.stl scale=1.00000 1.00000 1.00000
- link right_shoulder_x_link: geometry visual mesh filename=../meshes/stl/Texture.005.stl scale=1.00000 1.00000 1.00000; visual mesh filename=../meshes/stl/Texture.223.stl scale=1.00000 1.00000 1.00000
Joints:
- joint i01.head.eyeLeft_link_joint: limit lower=-0.17453 upper=0.17453 effort=0.00000 velocity=0.78540 -> lower=-0.78530 upper=0.78530 effort=0.00000 velocity=0.78540
- joint i01.head.eyeRight_link_joint: limit lower=-0.17453 upper=0.17453 effort=0.00000 velocity=0.78540 -> lower=-0.78530 upper=0.78530 effort=0.00000 velocity=0.78540

Commit message: evol(urdf): Update final I1 version
Signed-off-by: Mael-RABOT <mael.rabot@epitech.eu>

File: InMoov/urdf/InMoov.urdf (robot description, URDF)
Before this commit: robot InMoov, 55 links, 54 joints
Links:
- added link i01.head.eyeLeft.001_link
- added link i01.head.eyeRight.001_link
- added link i01.head.neck.001_link
- added link i01.head.rothead_link; visual mesh filename=../meshes/stl/Texture.013.stl scale=1.00000 1.00000 1.00000; visual mesh filename=../meshes/stl/Texture.068.stl scale=1.00000 1.00000 1.00000
Joints:
- added joint i01.head.eyeLeft.001_link_joint: type revolute, parent i01.head.rothead_link, child i01.head.eyeLeft.001_link, origin xyz=-1.08601 -0.29198 0.37576 rpy=0.00000 0.00000 -1.57080, axis 0.00000 0.00000 1.00000, limit lower=-0.34907 upper=0.34907 effort=0.00000 velocity=0.78540
- added joint i01.head.eyeRight.001_link_joint: type revolute, parent i01.head.rothead_link, child i01.head.eyeRight.001_link, origin xyz=-1.09644 0.29850 0.37576 rpy=-0.00000 -0.00000 -1.57080, axis 0.00000 0.00000 1.00000, limit lower=-0.34907 upper=0.34907 effort=0.00000 velocity=0.78540
- added joint i01.head.neck.001_link_joint: type revolute, parent torso_y_link, child i01.head.neck.001_link, origin xyz=0.00390 0.29817 4.29073 rpy=0.06589 -0.00000 -0.00000, axis 0.99994 0.00000 0.01111, limit lower=-0.34907 upper=0.34907 effort=0.00000 velocity=0.78540
- added joint i01.head.rothead_link_joint: type revolute, parent neck_link, child i01.head.rothead_link, origin xyz=0.00246 0.01503 0.24911 rpy=0.00000 -0.00000 1.57080, axis 0.00000 0.00000 1.00000, limit lower=-0.52360 upper=0.52360 effort=0.00000 velocity=0.78540
- joint Empty.002_link_joint: axis (none) -> 0.00000 0.00000 1.00000; limit (none) -> lower=0 upper=0 effort=0.00000 velocity=0.78540; type fixed -> continuous
- joint i01.head.eyeLeft_link_joint: origin xyz=0.29444 -1.07687 0.62487 rpy=0.00000 0.00000 -0.00000 -> xyz=0.00000 -0.00590 0.00000 rpy=0.00000 -0.00000 0.00000; parent neck_link -> i01.head.eyeLeft.001_link
- joint i01.head.eyeRight_link_joint: origin xyz=-0.29604 -1.08731 0.62487 rpy=0.00000 -0.00000 -0.00000 -> xyz=-0.00000 -0.00590 0.00000 rpy=0.00000 -0.00000 0.00000; parent neck_link -> i01.head.eyeRight.001_link
- joint i01.head.jaw_link_joint: origin xyz=-0.00876 -0.34673 0.57354 rpy=-0.00000 0.00000 -0.00000 -> xyz=-0.36176 0.01121 0.32442 rpy=-0.00000 -0.00000 -1.57080; parent neck_link -> i01.head.rothead_link
- joint i01.head.rollNeck_link_joint: axis (none) -> 0.00000 0.99994 0.01111; limit lower=0 upper=0 velocity=0.78540 -> lower=-0.34907 upper=0.34907 effort=0.00000 velocity=0.78540; origin xyz=0.00390 0.29788 4.29506 rpy=0.06589 -0.00000 -0.00000 -> xyz=0.00000 -0.00000 0.00435 rpy=-0.00000 0.00000 -0.00000; parent torso_y_link -> i01.head.neck.001_link; type floating -> revolute
