Commit message: fix(isaacsim): removing empty textures in urdf

File: InMoov-IsaacSim/urdf/InMoov.urdf (robot description, URDF)
Before this commit: robot InMoov, 59 links, 58 joints
Links:
- link left_shoulder_x_link: geometry visual mesh filename=../meshes/stl/Texture003.stl scale=1.00000 1.00000 1.00000; visual mesh filename=../meshes/stl/Texture254.stl scale=1.00000 1.00000 1.00000

Commit message: fix(isaacsim): renaming G.stl files

File: InMoov-IsaacSim/urdf/InMoov.urdf (robot description, URDF)
Before this commit: robot InMoov, 59 links, 58 joints
Links:
- link left_shoulder_z_link: geometry visual mesh filename=../meshes/stl/G564753.stl scale=1.00000 1.00000 1.00000; visual mesh filename=../meshes/stl/G564753_001.stl scale=1.00000 1.00000 1.00000
- link right_shoulder_z_link: geometry visual mesh filename=../meshes/stl/G566220.stl scale=1.00000 1.00000 1.00000; visual mesh filename=../meshes/stl/G566220_001.stl scale=1.00000 1.00000 1.00000

Commit message: fix(isaacsim): removing empty G.stl files

File: InMoov-IsaacSim/urdf/InMoov.urdf (robot description, URDF)
Before this commit: robot InMoov, 59 links, 58 joints
Links:
- link right_shoulder_z_link: geometry visual mesh filename=../meshes/stl/G566220.stl scale=1.00000 1.00000 1.00000; visual mesh filename=../meshes/stl/G566220_001.stl scale=1.00000 1.00000 1.00000
