Commit message: evol(archi): applied standard urdf package structure
Signed-off-by: Charles Madjeri <charles@madjeri.com>

File: description/urdf/inmoov.urdf.xacro (robot description, xacro)
@@ -5,8 +5,8 @@
   <xacro:arg name="use_gazebo_sim" default="false"/>
   <xacro:arg name="controller_config" default=""/>
-  <xacro:property name="mesh_dir" value="file://$(arg base_path)/meshes/dae"/>
+  <xacro:property name="mesh_dir" value="file://$(arg base_path)/robot_description/meshes/dae"/>
   <xacro:property name="use_gazebo_sim" value="$(arg use_gazebo_sim)"/>
   <!-- Import inmoov physical description (urdf) macro (uses use_gazebo_sim for heavy stand in sim) -->
-  <xacro:include filename="../3dmodel/robot_description.urdf.xacro"/>
+  <xacro:include filename="../robot_description/urdf/robot_description.urdf.xacro"/>
   <!-- Import inmoov ros2_control description (use_gazebo_sim switches to gz_ros2_control in Gazebo launch) -->
   <xacro:include filename="../ros2_control/inmoov_ros2_control.xacro" />
