Commit message: feat(urdf): compilation of the xacro into a standalone urdf for dae, renaming inmoov-isaacsim to inmoov-stl

File: description/ros2_control/inmoov_ros2_control.xacro (robot description, xacro)
@@ -3,4 +3,5 @@
 <robot xmlns:xacro="http://www.ros.org/wiki/xacro" name="inmoov" version="1.0">
   <xacro:arg name="use_gazebo_sim" default="false" />
+  <xacro:arg name="use_mock_hardware" default="false" />
   <ros2_control name="LucyHardwareLeftArm" type="system">
       <hardware>
@@ -9,7 +10,12 @@
           </xacro:if>
           <xacro:unless value="$(arg use_gazebo_sim)">
-            <plugin>lucy_ros2_control/LucySystemHardware</plugin>
-            <param name="publisher_topic">actuators/left_arm</param>
-            <param name="node_name">lucy_hardware_interface_left_arm</param>
+            <xacro:if value="$(arg use_mock_hardware)">
+              <plugin>mock_components/GenericSystem</plugin>
+            </xacro:if>
+            <xacro:unless value="$(arg use_mock_hardware)">
+              <plugin>lucy_ros2_control/LucySystemHardware</plugin>
+              <param name="publisher_topic">actuators/left_arm</param>
+              <param name="node_name">lucy_hardware_interface_left_arm</param>
+            </xacro:unless>
           </xacro:unless>
       </hardware>
@@ -17,10 +23,10 @@
           <param name="virtual_pin">0</param>
           <param name="servo_type">270</param>
-          <param name="offset_deg">0.0</param>
-          <param name="direction">1</param>
-          <param name="scale">1.0</param>
-          <param name="servo_min_deg">0.0</param>
-          <param name="servo_max_deg">270.0</param>
-          <param name="servo_default_deg">135.0</param>
+          <param name="offset_deg">0</param>
+          <param name="direction">1</param>
+          <param name="scale">1</param>
+          <param name="servo_min_deg">0</param>
+          <param name="servo_max_deg">270</param>
+          <param name="servo_default_deg">135</param>
           <command_interface name="position" />
           <state_interface name="position" />
@@ -29,10 +35,10 @@
           <param name="virtual_pin">1</param>
           <param name="servo_type">270</param>
-          <param name="offset_deg">0.0</param>
-          <param name="direction">1</param>
-          <param name="scale">1.0</param>
-          <param name="servo_min_deg">0.0</param>
-          <param name="servo_max_deg">270.0</param>
-          <param name="servo_default_deg">135.0</param>
+          <param name="offset_deg">0</param>
+          <param name="direction">1</param>
+          <param name="scale">1</param>
+          <param name="servo_min_deg">0</param>
+          <param name="servo_max_deg">270</param>
+          <param name="servo_default_deg">135</param>
           <command_interface name="position" />
           <state_interface name="position" />
@@ -41,10 +47,10 @@
           <param name="virtual_pin">2</param>
           <param name="servo_type">270</param>
-          <param name="offset_deg">0.0</param>
-          <param name="direction">1</param>
-          <param name="scale">1.0</param>
-          <param name="servo_min_deg">0.0</param>
-          <param name="servo_max_deg">270.0</param>
-          <param name="servo_default_deg">90.0</param>
+          <param name="offset_deg">0</param>
+          <param name="direction">1</param>
+          <param name="scale">1</param>
+          <param name="servo_min_deg">0</param>
+          <param name="servo_max_deg">270</param>
+          <param name="servo_default_deg">90</param>
           <command_interface name="position" />
           <state_interface name="position" />
@@ -53,10 +59,10 @@
           <param name="virtual_pin">3</param>
           <param name="servo_type">300</param>
-          <param name="offset_deg">0.0</param>
-          <param name="direction">1</param>
-          <param name="scale">1.0</param>
-          <param name="servo_min_deg">0.0</param>
-          <param name="servo_max_deg">150.0</param>
-          <param name="servo_default_deg">50.0</param>
+          <param name="offset_deg">0</param>
+          <param name="direction">1</param>
+          <param name="scale">1</param>
+          <param name="servo_min_deg">0</param>
+          <param name="servo_max_deg">150</param>
+          <param name="servo_default_deg">50</param>
           <command_interface name="position" />
           <state_interface name="position" />
@@ -65,10 +71,10 @@
           <param name="virtual_pin">4</param>
           <param name="servo_type">300</param>
-          <param name="offset_deg">0.0</param>
-          <param name="direction">1</param>
-          <param name="scale">1.0</param>
-          <param name="servo_min_deg">0.0</param>
-          <param name="servo_max_deg">150.0</param>
-          <param name="servo_default_deg">50.0</param>
+          <param name="offset_deg">0</param>
+          <param name="direction">1</param>
+          <param name="scale">1</param>
+          <param name="servo_min_deg">0</param>
+          <param name="servo_max_deg">150</param>
+          <param name="servo_default_deg">50</param>
           <command_interface name="position" />
           <state_interface name="position" />
@@ -77,10 +83,10 @@
           <param name="virtual_pin">5</param>
           <param name="servo_type">300</param>
-          <param name="offset_deg">0.0</param>
-          <param name="direction">1</param>
-          <param name="scale">1.0</param>
-          <param name="servo_min_deg">0.0</param>
-          <param name="servo_max_deg">150.0</param>
-          <param name="servo_default_deg">50.0</param>
+          <param name="offset_deg">0</param>
+          <param name="direction">1</param>
+          <param name="scale">1</param>
+          <param name="servo_min_deg">0</param>
+          <param name="servo_max_deg">150</param>
+          <param name="servo_default_deg">50</param>
           <command_interface name="position" />
           <state_interface name="position" />
@@ -89,10 +95,10 @@
           <param name="virtual_pin">6</param>
           <param name="servo_type">300</param>
-          <param name="offset_deg">0.0</param>
-          <param name="direction">1</param>
-          <param name="scale">1.0</param>
-          <param name="servo_min_deg">0.0</param>
-          <param name="servo_max_deg">150.0</param>
-          <param name="servo_default_deg">50.0</param>
+          <param name="offset_deg">0</param>
+          <param name="direction">1</param>
+          <param name="scale">1</param>
+          <param name="servo_min_deg">0</param>
+          <param name="servo_max_deg">150</param>
+          <param name="servo_default_deg">50</param>
           <command_interface name="position" />
           <state_interface name="position" />
@@ -101,10 +107,10 @@
           <param name="virtual_pin">7</param>
           <param name="servo_type">300</param>
-          <param name="offset_deg">0.0</param>
-          <param name="direction">1</param>
-          <param name="scale">1.0</param>
-          <param name="servo_min_deg">0.0</param>
-          <param name="servo_max_deg">150.0</param>
-          <param name="servo_default_deg">50.0</param>
+          <param name="offset_deg">0</param>
+          <param name="direction">1</param>
+          <param name="scale">1</param>
+          <param name="servo_min_deg">0</param>
+          <param name="servo_max_deg">150</param>
+          <param name="servo_default_deg">50</param>
           <command_interface name="position" />
           <state_interface name="position" />
@@ -113,10 +119,10 @@
           <param name="virtual_pin">8</param>
           <param name="servo_type">300</param>
-          <param name="offset_deg">0.0</param>
-          <param name="direction">1</param>
-          <param name="scale">1.0</param>
-          <param name="servo_min_deg">0.0</param>
-          <param name="servo_max_deg">150.0</param>
-          <param name="servo_default_deg">50.0</param>
+          <param name="offset_deg">0</param>
+          <param name="direction">1</param>
+          <param name="scale">1</param>
+          <param name="servo_min_deg">0</param>
+          <param name="servo_max_deg">150</param>
+          <param name="servo_default_deg">50</param>
           <command_interface name="position" />
           <state_interface name="position" />
@@ -129,7 +135,12 @@
           </xacro:if>
           <xacro:unless value="$(arg use_gazebo_sim)">
-            <plugin>lucy_ros2_control/LucySystemHardware</plugin>
-            <param name="publisher_topic">actuators/right_arm</param>
-            <param name="node_name">lucy_hardware_interface_right_arm</param>
+            <xacro:if value="$(arg use_mock_hardware)">
+              <plugin>mock_components/GenericSystem</plugin>
+            </xacro:if>
+            <xacro:unless value="$(arg use_mock_hardware)">
+              <plugin>lucy_ros2_control/LucySystemHardware</plugin>
+              <param name="publisher_topic">actuators/right_arm</param>
+              <param name="node_name">lucy_hardware_interface_right_arm</param>
+            </xacro:unless>
           </xacro:unless>
       </hardware>
@@ -137,10 +148,10 @@
           <param name="virtual_pin">0</param>
           <param name="servo_type">270</param>
-          <param name="offset_deg">0.0</param>
-          <param name="direction">1</param>
-          <param name="scale">1.0</param>
-          <param name="servo_min_deg">155.0</param>
-          <param name="servo_max_deg">165.0</param>
-          <param name="servo_default_deg">160.0</param>
+          <param name="offset_deg">0</param>
+          <param name="direction">1</param>
+          <param name="scale">1</param>
+          <param name="servo_min_deg">155</param>
+          <param name="servo_max_deg">165</param>
+          <param name="servo_default_deg">160</param>
           <command_interface name="position" />
           <state_interface name="position" />
@@ -149,10 +160,10 @@
           <param name="virtual_pin">1</param>
           <param name="servo_type">270</param>
-          <param name="offset_deg">0.0</param>
-          <param name="direction">1</param>
-          <param name="scale">1.0</param>
-          <param name="servo_min_deg">140.0</param>
-          <param name="servo_max_deg">180.0</param>
-          <param name="servo_default_deg">180.0</param>
+          <param name="offset_deg">0</param>
+          <param name="direction">1</param>
+          <param name="scale">1</param>
+          <param name="servo_min_deg">140</param>
+          <param name="servo_max_deg">180</param>
+          <param name="servo_default_deg">180</param>
           <command_interface name="position" />
           <state_interface name="position" />
@@ -161,10 +172,10 @@
           <param name="virtual_pin">2</param>
           <param name="servo_type">270</param>
-          <param name="offset_deg">0.0</param>
-          <param name="direction">1</param>
-          <param name="scale">1.0</param>
-          <param name="servo_min_deg">100.0</param>
-          <param name="servo_max_deg">110.0</param>
-          <param name="servo_default_deg">100.0</param>
+          <param name="offset_deg">0</param>
+          <param name="direction">1</param>
+          <param name="scale">1</param>
+          <param name="servo_min_deg">100</param>
+          <param name="servo_max_deg">110</param>
+          <param name="servo_default_deg">100</param>
           <command_interface name="position" />
           <state_interface name="position" />
@@ -173,10 +184,10 @@
           <param name="virtual_pin">3</param>
           <param name="servo_type">300</param>
-          <param name="offset_deg">0.0</param>
-          <param name="direction">1</param>
-          <param name="scale">1.0</param>
-          <param name="servo_min_deg">0.0</param>
-          <param name="servo_max_deg">230.0</param>
-          <param name="servo_default_deg">150.0</param>
+          <param name="offset_deg">0</param>
+          <param name="direction">1</param>
+          <param name="scale">1</param>
+          <param name="servo_min_deg">0</param>
+          <param name="servo_max_deg">230</param>
+          <param name="servo_default_deg">150</param>
           <command_interface name="position" />
           <state_interface name="position" />
@@ -185,10 +196,10 @@
           <param name="virtual_pin">4</param>
           <param name="servo_type">300</param>
-          <param name="offset_deg">0.0</param>
-          <param name="direction">1</param>
-          <param name="scale">1.0</param>
-          <param name="servo_min_deg">36.0</param>
-          <param name="servo_max_deg">150.0</param>
-          <param name="servo_default_deg">36.0</param>
+          <param name="offset_deg">0</param>
+          <param name="direction">1</param>
+          <param name="scale">1</param>
+          <param name="servo_min_deg">36</param>
+          <param name="servo_max_deg">150</param>
+          <param name="servo_default_deg">36</param>
           <command_interface name="position" />
           <state_interface name="position" />
@@ -197,10 +208,10 @@
           <param name="virtual_pin">5</param>
           <param name="servo_type">300</param>
-          <param name="offset_deg">0.0</param>
-          <param name="direction">1</param>
-          <param name="scale">1.0</param>
-          <param name="servo_min_deg">16.0</param>
-          <param name="servo_max_deg">150.0</param>
-          <param name="servo_default_deg">16.0</param>
+          <param name="offset_deg">0</param>
+          <param name="direction">1</param>
+          <param name="scale">1</param>
+          <param name="servo_min_deg">16</param>
+          <param name="servo_max_deg">150</param>
+          <param name="servo_default_deg">16</param>
           <command_interface name="position" />
           <state_interface name="position" />
@@ -209,10 +220,10 @@
           <param name="virtual_pin">6</param>
           <param name="servo_type">300</param>
-          <param name="offset_deg">0.0</param>
-          <param name="direction">1</param>
-          <param name="scale">1.0</param>
-          <param name="servo_min_deg">21.0</param>
-          <param name="servo_max_deg">150.0</param>
-          <param name="servo_default_deg">21.0</param>
+          <param name="offset_deg">0</param>
+          <param name="direction">1</param>
+          <param name="scale">1</param>
+          <param name="servo_min_deg">21</param>
+          <param name="servo_max_deg">150</param>
+          <param name="servo_default_deg">21</param>
           <command_interface name="position" />
           <state_interface name="position" />
@@ -221,10 +232,10 @@
           <param name="virtual_pin">7</param>
           <param name="servo_type">300</param>
-          <param name="offset_deg">0.0</param>
-          <param name="direction">1</param>
-          <param name="scale">1.0</param>
-          <param name="servo_min_deg">33.0</param>
-          <param name="servo_max_deg">150.0</param>
-          <param name="servo_default_deg">33.0</param>
+          <param name="offset_deg">0</param>
+          <param name="direction">1</param>
+          <param name="scale">1</param>
+          <param name="servo_min_deg">33</param>
+          <param name="servo_max_deg">150</param>
+          <param name="servo_default_deg">33</param>
           <command_interface name="position" />
           <state_interface name="position" />
@@ -233,10 +244,10 @@
           <param name="virtual_pin">8</param>
           <param name="servo_type">300</param>
-          <param name="offset_deg">0.0</param>
-          <param name="direction">1</param>
-          <param name="scale">1.0</param>
-          <param name="servo_min_deg">30.0</param>
-          <param name="servo_max_deg">150.0</param>
-          <param name="servo_default_deg">30.0</param>
+          <param name="offset_deg">0</param>
+          <param name="direction">1</param>
+          <param name="scale">1</param>
+          <param name="servo_min_deg">30</param>
+          <param name="servo_max_deg">150</param>
+          <param name="servo_default_deg">30</param>
           <command_interface name="position" />
           <state_interface name="position" />
@@ -249,7 +260,12 @@
           </xacro:if>
           <xacro:unless value="$(arg use_gazebo_sim)">
-            <plugin>lucy_ros2_control/LucySystemHardware</plugin>
-            <param name="publisher_topic">actuators/torso</param>
-            <param name="node_name">lucy_hardware_interface_torso_head</param>
+            <xacro:if value="$(arg use_mock_hardware)">
+              <plugin>mock_components/GenericSystem</plugin>
+            </xacro:if>
+            <xacro:unless value="$(arg use_mock_hardware)">
+              <plugin>lucy_ros2_control/LucySystemHardware</plugin>
+              <param name="publisher_topic">actuators/torso</param>
+              <param name="node_name">lucy_hardware_interface_torso_head</param>
+            </xacro:unless>
           </xacro:unless>
       </hardware>
@@ -257,10 +273,10 @@
           <param name="virtual_pin">0</param>
           <param name="servo_type">270</param>
-          <param name="offset_deg">0.0</param>
-          <param name="direction">1</param>
-          <param name="scale">1.0</param>
-          <param name="servo_min_deg">0.0</param>
-          <param name="servo_max_deg">270.0</param>
-          <param name="servo_default_deg">0.0</param>
+          <param name="offset_deg">0</param>
+          <param name="direction">1</param>
+          <param name="scale">1</param>
+          <param name="servo_min_deg">0</param>
+          <param name="servo_max_deg">270</param>
+          <param name="servo_default_deg">0</param>
           <command_interface name="position" />
           <state_interface name="position" />
@@ -269,10 +285,22 @@
           <param name="virtual_pin">1</param>
           <param name="servo_type">270</param>
-          <param name="offset_deg">0.0</param>
-          <param name="direction">1</param>
-          <param name="scale">1.0</param>
-          <param name="servo_min_deg">0.0</param>
-          <param name="servo_max_deg">270.0</param>
-          <param name="servo_default_deg">0.0</param>
+          <param name="offset_deg">0</param>
+          <param name="direction">1</param>
+          <param name="scale">1</param>
+          <param name="servo_min_deg">0</param>
+          <param name="servo_max_deg">270</param>
+          <param name="servo_default_deg">0</param>
+          <command_interface name="position" />
+          <state_interface name="position" />
+      </joint>
+      <joint name="i01.torso.topStom_link_joint">
+          <param name="virtual_pin">2</param>
+          <param name="servo_type">270</param>
+          <param name="offset_deg">0</param>
+          <param name="direction">1</param>
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
Commit message: fix(urdf): compiled urdf should be next to the xacro parent

File: description/ros2_control/inmoov_ros2_control.xacro (robot description, xacro)
@@ -306,4 +306,16 @@
           <state_interface name="position" />
       </joint>
+      <joint name="i01.torso.midStom_link_joint">
+          <param name="virtual_pin">3</param>
+          <param name="servo_type">270</param>
+          <param name="offset_deg">0</param>
+          <param name="direction">1</param>
+          <param name="scale">1</param>
+          <param name="servo_min_deg">0</param>
+          <param name="servo_max_deg">270</param>
+          <param name="servo_default_deg">135</param>
+          <command_interface name="position" />
+          <state_interface name="position" />
+      </joint>
   </ros2_control>
 </robot>
