Commit message: Make the Gazebo GUI work on macOS and keep the robot upright
Same three macOS simulator faults as inmoov_urdf, which thais_urdf shares
verbatim (same physics xacro, same launch shape).

1. gz sim exits(-1) when given neither -s nor -g, because Cocoa requires the Qt
   GUI on the main thread (gazebosim/gz-sim#44). The launch passed plain
   "-r <world>", so the server died at once. On Darwin run the server with -s
   and start `gz sim -g` as a second, delayed process.

2. <static>true</static> on a link does not survive urdf->sdf conversion, and
   the robot spawned at -z 0.5 in midair, so gravity toppled it. Anchor
   base_node to a `world` link with a fixed joint and spawn at -z 0.0. Gated
   behind use_gazebo_sim:=true, so the real/mock TF tree is unaffected
   (verified: 0 occurrences in the non-sim description).

3. filename="libmock_sensor.so" is hardcoded; the plugin builds as
   libmock_sensor.dylib on macOS. A bare "mock_sensor" lets Gazebo resolve the
   platform extension.

Builds clean and the sim description resolves; the GUI itself was verified on
inmoov_urdf, which is the robot package in use here.

File: description/gazebo/inmoov_gazebo_physics.xacro (robot description, xacro)
@@ -13,4 +13,18 @@
 <robot xmlns:xacro="http://www.ros.org/wiki/xacro">
   <!-- Fix entire stand to the world so the robot does not fall (gz-sim may still move root; heavy mass in URDF is fallback). -->
+  <!-- Anchor the stand to the world so the robot does not fall over.
+       <gazebo reference="..."><static>true</static></gazebo> does not survive
+       urdf->sdf conversion: sdformat only honours <static> on the model, not on
+       a link, so the stand stayed dynamic and gravity toppled the robot. A fixed
+       joint to a `world` link is the conversion-stable way to pin the base, and
+       leaves every upper-body joint (torso, neck, arms, fingers) free to move.
+       This file is included only under use_gazebo_sim:=true, so the extra link
+       never reaches the real/mock-hardware description or its TF tree. -->
+  <link name="world"/>
+  <joint name="world_to_base_node" type="fixed">
+    <parent link="world"/>
+    <child link="base_node"/>
+    <origin xyz="0 0 0.02" rpy="0 0 0"/>
+  </joint>
   <gazebo reference="base_node">
     <static>true</static>

Commit message: evol(package): sync thais_urdf with inmoov_urdf jazzy and sim stack while keeping thais hardware presets

File: description/gazebo/inmoov_gazebo_physics.xacro (robot description, xacro)
@@ -3,7 +3,7 @@
      use_gazebo_sim:=true. This file is pure simulation tuning: world
      anchoring, friction, contact stiffness, and self-collision flags.
-     The gz_ros2_control plugin itself lives next door in
-     description/ros2_control/inmoov_gz_ros2_control.xacro because it is the
-     ros2_control bridge into Gazebo, not a physics property.
+     The gz_ros2_control plugin itself lives next door in the generated
+     description/gazebo/gazebo.xacro because it is the ros2_control bridge
+     into Gazebo (and carries the camera sensors), not a physics property.
      Collision strategy: every URDF link reuses its visual mesh as the
      collision mesh (see scripts/inject_collisions.py). The macros below only
@@ -12,8 +12,18 @@
      enables it with friction tuned for grasping. -->
 <robot xmlns:xacro="http://www.ros.org/wiki/xacro">
-  <!-- Fix entire stand to the world so the robot does not fall (gz-sim may still move root; heavy mass in URDF is fallback). -->
-  <gazebo reference="base_node">
-    <static>true</static>
-  </gazebo>
+  <!-- Anchor the stand to the world so the robot does not fall over.
+       <gazebo reference="..."><static>true</static></gazebo> does not survive
+       urdf->sdf conversion: sdformat only honours <static> on the model, not on
+       a link, so the stand stayed dynamic and gravity toppled the robot. A fixed
+       joint to a `world` link is the conversion-stable way to pin the base, and
+       leaves every upper-body joint (torso, neck, arms, fingers) free to move.
+       This file is included only under use_gazebo_sim:=true, so the extra link
+       never reaches the real/mock-hardware description or its TF tree. -->
+  <link name="world"/>
+  <joint name="world_to_base_node" type="fixed">
+    <parent link="world"/>
+    <child link="base_node"/>
+    <origin xyz="0 0 0.02" rpy="0 0 0"/>
+  </joint>
   <gazebo reference="stand_link">
     <static>true</static>

File: description/urdf/inmoov.urdf.xacro (robot description, xacro)
@@ -15,5 +15,7 @@
   <!-- Import inmoov physical description (urdf) macro (uses use_gazebo_sim for heavy stand in sim) -->
   <xacro:include filename="../robot_description/urdf/robot_description.urdf.xacro"/>
-  <!-- Import inmoov ros2_control description (use_gazebo_sim switches to gz_ros2_control in Gazebo launch).
+  <!-- Import inmoov ros2_control description for real/mock hardware only.
+       In Gazebo (use_gazebo_sim:=true) the generated gazebo/gazebo.xacro provides the
+       gz_ros2_control system instead, so skip this include to avoid double registration.
        Filename comes from the generated_files config so the generator, pipeline and launches agree. -->
   <!-- Import inmoov ros2_control description (use_gazebo_sim switches to gz_ros2_control in Gazebo launch) -->
@@ -24,7 +26,7 @@
          - gazebo/inmoov_gazebo_physics.xacro    physics + surface tuning
                                                  (static stand, friction, self_collide, kp/kd)
-         - ros2_control/inmoov_gz_ros2_control.xacro
-                                                 gz_ros2_control plugin so the same
-                                                 controllers drive simulated joints -->
+         - gazebo/gazebo.xacro                   generated gz_ros2_control plugin +
+                                                 camera sensors so the same controllers
+                                                 drive simulated joints -->
   <xacro:if value="$(arg use_gazebo_sim)">
     <xacro:include filename="../gazebo/inmoov_gazebo_physics.xacro"/>
